Commit message: Updated locomotion ready for PACE results

File: source/BDXR/data/Robots/BDXR/URDF.urdf (robot description, URDF)
Before this commit: robot URDF, 77 links, 76 joints
Links:
- link Back_Support: mass 1.4345660747046487 -> 0.1; geometry collision mesh filename=./meshes/Back_Support.stl scale=0.001 0.001 0.001; visual mesh filename=./meshes/Back_Support.stl scale=0.001 0.001 0.001
- link Base_Top_Clamp: mass 0.34279762697415633 -> 0.044; geometry collision mesh filename=./meshes/Base_Top_Clamp.stl scale=0.001 0.001 0.001; visual mesh filename=./meshes/Base_Top_Clamp.stl scale=0.001 0.001 0.001
- link Battery: mass 7.946971853050029 -> 1.25; geometry collision mesh filename=./meshes/Battery.stl scale=0.001 0.001 0.001; visual mesh filename=./meshes/Battery.stl scale=0.001 0.001 0.001
- link Battery_Holder: mass 1.2003975073649495 -> 0.18; geometry collision mesh filename=./meshes/Battery_Holder.stl scale=0.001 0.001 0.001; visual mesh filename=./meshes/Battery_Holder.stl scale=0.001 0.001 0.001
- link Bottom_Cover: mass 0.2325777541774406 -> 0.1; geometry collision mesh filename=./meshes/Bottom_Cover.stl scale=0.001 0.001 0.001; visual mesh filename=./meshes/Bottom_Cover.stl scale=0.001 0.001 0.001
- link Camera_Mount: mass 0.23780328755101082 -> 0.04; geometry collision mesh filename=./meshes/Camera_Mount.stl scale=0.001 0.001 0.001; visual mesh filename=./meshes/Camera_Mount.stl scale=0.001 0.001 0.001
- link Face: mass 0.3825323982770003 -> 0.1; geometry collision mesh filename=./meshes/Face.stl scale=0.001 0.001 0.001; visual mesh filename=./meshes/Face.stl scale=0.001 0.001 0.001
- link Front_Cover: mass 3.016585112031044 -> 0.2; geometry collision mesh filename=./meshes/Front_Cover.stl scale=0.001 0.001 0.001; visual mesh filename=./meshes/Front_Cover.stl scale=0.001 0.001 0.001
- link Front_Grill: mass 0.12278343435530116 -> 0.01; geometry collision mesh filename=./meshes/Front_Grill.stl scale=0.001 0.001 0.001; visual mesh filename=./meshes/Front_Grill.stl scale=0.001 0.001 0.001
- link Front_Support: mass 1.3644492060488889 -> 0.15; geometry collision mesh filename=./meshes/Front_Support.stl scale=0.001 0.001 0.001; visual mesh filename=./meshes/Front_Support.stl scale=0.001 0.001 0.001
- link Head_Base_Plate: mass 0.7026538517747032 -> 0.24; geometry collision mesh filename=./meshes/Head_Base_Plate.stl scale=0.001 0.001 0.001; visual mesh filename=./meshes/Head_Base_Plate.stl scale=0.001 0.001 0.001
- link Head_Pitch_Motor: geometry collision mesh filename=./meshes/Head_Pitch_Motor.stl scale=0.001 0.001 0.001; visual mesh filename=./meshes/Head_Pitch_Motor.stl scale=0.001 0.001 0.001
- link Head_Pitch_Motor_Support: mass 0.3978591096412742 -> 0.08; geometry collision mesh filename=./meshes/Head_Pitch_Motor_Support.stl scale=0.001 0.001 0.001; visual mesh filename=./meshes/Head_Pitch_Motor_Support.stl scale=0.001 0.001 0.001
- link Head_Rear_Cover: mass 2.1083250067116728 -> 0.1; geometry collision mesh filename=./meshes/Head_Rear_Cover.stl scale=0.001 0.001 0.001; visual mesh filename=./meshes/Head_Rear_Cover.stl scale=0.001 0.001 0.001
- link Head_Roll_Connector: mass 0.1909286096033978 -> 0.05; geometry collision mesh filename=./meshes/Head_Roll_Connector.stl scale=0.001 0.001 0.001; visual mesh filename=./meshes/Head_Roll_Connector.stl scale=0.001 0.001 0.001
- link Head_Roll_Motor: geometry collision mesh filename=./meshes/Head_Roll_Motor.stl scale=0.001 0.001 0.001; visual mesh filename=./meshes/Head_Roll_Motor.stl scale=0.001 0.001 0.001
- link Head_Roll_Motor_Mount: mass 0.42782888507946565 -> 0.08; geometry collision mesh filename=./meshes/Head_Roll_Motor_Mount.stl scale=0.001 0.001 0.001; visual mesh filename=./meshes/Head_Roll_Motor_Mount.stl scale=0.001 0.001 0.001
- link Head_Yaw_Motor: geometry collision mesh filename=./meshes/Head_Yaw_Motor.stl scale=0.001 0.001 0.001; visual mesh filename=./meshes/Head_Yaw_Motor.stl scale=0.001 0.001 0.001
- link Left_Ankle_Cover: mass 0.10517582367621381 -> 0.01; geometry collision mesh filename=./meshes/Left_Ankle_Cover.stl scale=0.001 0.001 0.001; visual mesh filename=./meshes/Left_Ankle_Cover.stl scale=0.001 0.001 0.001
- link Left_Ankle_Motor: geometry collision mesh filename=./meshes/Left_Ankle_Motor.stl scale=0.001 0.001 0.001; visual mesh filename=./meshes/Left_Ankle_Motor.stl scale=0.001 0.001 0.001
- link Left_Cable_Support: mass 0.4093453218387253 -> 0.08; geometry collision mesh filename=./meshes/Left_Cable_Support.stl scale=0.001 0.001 0.001; visual mesh filename=./meshes/Left_Cable_Support.stl scale=0.001 0.001 0.001
- link Left_Ear: mass 0.08364465059570073 -> 0.01; geometry collision mesh filename=./meshes/Left_Ear.stl scale=0.001 0.001 0.001; visual mesh filename=./meshes/Left_Ear.stl scale=0.001 0.001 0.001
- link Left_Eye: mass 0.1126202923319544 -> 0.02; geometry collision mesh filename=./meshes/Left_Eye.stl scale=0.001 0.001 0.001; visual mesh filename=./meshes/Left_Eye.stl scale=0.001 0.001 0.001
- link Left_Foot: mass 1.8791037125473142 -> 0.22; geometry collision mesh filename=./meshes/Left_Foot.stl scale=0.001 0.001 0.001; visual mesh filename=./meshes/Left_Foot.stl scale=0.001 0.001 0.001
- link Left_Foot_Cover: mass 0.2778877451208695 -> 0.02; geometry collision mesh filename=./meshes/Left_Foot_Cover.stl scale=0.001 0.001 0.001; visual mesh filename=./meshes/Left_Foot_Cover.stl scale=0.001 0.001 0.001
- link Left_Foot_Pad: mass 0.8235307524446849 -> 0.08; geometry collision mesh filename=./meshes/Left_Foot_Pad.stl scale=0.001 0.001 0.001; visual mesh filename=./meshes/Left_Foot_Pad.stl scale=0.001 0.001 0.001
- link Left_Front_Cover: mass 0.5492461618694918 -> 0.1; geometry collision mesh filename=./meshes/Left_Front_Cover.stl scale=0.001 0.001 0.001; visual mesh filename=./meshes/Left_Front_Cover.stl scale=0.001 0.001 0.001
- link Left_Head_Support: mass 0.15134820623495676 -> 0.04; geometry collision mesh filename=./meshes/Left_Head_Support.stl scale=0.001 0.001 0.001; visual mesh filename=./meshes/Left_Head_Support.stl scale=0.001 0.001 0.001
- link Left_Hip_Bottom_Holder: mass 0.44482107671145055 -> 0.075; geometry collision mesh filename=./meshes/Left_Hip_Bottom_Holder.stl scale=0.001 0.001 0.001; visual mesh filename=./meshes/Left_Hip_Bottom_Holder.stl scale=0.001 0.001 0.001
- link Left_Hip_Pitch_Motor: mass 0.880 -> 0.920; geometry collision mesh filename=./meshes/Left_Hip_Pitch_Motor.stl scale=0.001 0.001 0.001; visual mesh filename=./meshes/Left_Hip_Pitch_Motor.stl scale=0.001 0.001 0.001
- link Left_Hip_Roll_Connector: mass 0.28535022457844034 -> 0.1; geometry collision mesh filename=./meshes/Left_Hip_Roll_Connector.stl scale=0.001 0.001 0.001; visual mesh filename=./meshes/Left_Hip_Roll_Connector.stl scale=0.001 0.001 0.001
- link Left_Hip_Roll_Motor: mass 0.880 -> 0.920; geometry collision mesh filename=./meshes/Left_Hip_Roll_Motor.stl scale=0.001 0.001 0.001; visual mesh filename=./meshes/Left_Hip_Roll_Motor.stl scale=0.001 0.001 0.001
- link Left_Hip_Top_Holder: mass 0.6080984706410992 -> 0.08; geometry collision mesh filename=./meshes/Left_Hip_Top_Holder.stl scale=0.001 0.001 0.001; visual mesh filename=./meshes/Left_Hip_Top_Holder.stl scale=0.001 0.001 0.001
- link Left_Hip_Yaw_Motor: mass 0.880 -> 0.920; geometry collision mesh filename=./meshes/Left_Hip_Yaw_Motor.stl scale=0.001 0.001 0.001; visual mesh filename=./meshes/Left_Hip_Yaw_Motor.stl scale=0.001 0.001 0.001
- link Left_Hip_Yaw_Support: mass 0.8129334554771345 -> 0.08; geometry collision mesh filename=./meshes/Left_Hip_Yaw_Support.stl scale=0.001 0.001 0.001; visual mesh filename=./meshes/Left_Hip_Yaw_Support.stl scale=0.001 0.001 0.001
- link Left_Holder: mass 0.37776469464112955 -> 0.08; geometry collision mesh filename=./meshes/Left_Holder.stl scale=0.001 0.001 0.001; visual mesh filename=./meshes/Left_Holder.stl scale=0.001 0.001 0.001
- link Left_Knee_Motor: mass 0.880 -> 0.920; geometry collision mesh filename=./meshes/Left_Knee_Motor.stl scale=0.001 0.001 0.001; visual mesh filename=./meshes/Left_Knee_Motor.stl scale=0.001 0.001 0.001
- link Left_Lower_Leg: mass 2.8649012995453993 -> 0.33; geometry collision mesh filename=./meshes/Left_Lower_Leg.stl scale=0.001 0.001 0.001; visual mesh filename=./meshes/Left_Lower_Leg.stl scale=0.001 0.001 0.001
- link Left_Lower_Leg_Cover: mass 0.6798560279056552 -> 0.057; geometry collision mesh filename=./meshes/Left_Lower_Leg_Cover.stl scale=0.001 0.001 0.001; visual mesh filename=./meshes/Left_Lower_Leg_Cover.stl scale=0.001 0.001 0.001
- link Left_Top_Cover: mass 0.30626446288176407 -> 0.03; geometry collision mesh filename=./meshes/Left_Top_Cover.stl scale=0.001 0.001 0.001; visual mesh filename=./meshes/Left_Top_Cover.stl scale=0.001 0.001 0.001
- link Left_Upper_Leg: mass 4.1882983071068365 -> 0.5; geometry collision mesh filename=./meshes/Left_Upper_Leg.stl scale=0.001 0.001 0.001; visual mesh filename=./meshes/Left_Upper_Leg.stl scale=0.001 0.001 0.001
- link Left_Upper_Leg_Cover: mass 0.4710868540250967 -> 0.075; geometry collision mesh filename=./meshes/Left_Upper_Leg_Cover.stl scale=0.001 0.001 0.001; visual mesh filename=./meshes/Left_Upper_Leg_Cover.stl scale=0.001 0.001 0.001
- link Left_Upper_Leg_Detail: mass 0.0367883220982521 -> 0.01; geometry collision mesh filename=./meshes/Left_Upper_Leg_Detail.stl scale=0.001 0.001 0.001; visual mesh filename=./meshes/Left_Upper_Leg_Detail.stl scale=0.001 0.001 0.001
- link Neck: mass 1.3919244642510382 -> 0.2; geometry collision mesh filename=./meshes/Neck.stl scale=0.001 0.001 0.001; visual mesh filename=./meshes/Neck.stl scale=0.001 0.001 0.001
- link Neck_Motor: geometry collision mesh filename=./meshes/Neck_Motor.stl scale=0.001 0.001 0.001; visual mesh filename=./meshes/Neck_Motor.stl scale=0.001 0.001 0.001
- link Rear_Antenna_Box: mass 0.4309225889234217 -> 0.1; geometry collision mesh filename=./meshes/Rear_Antenna_Box.stl scale=0.001 0.001 0.001; visual mesh filename=./meshes/Rear_Antenna_Box.stl scale=0.001 0.001 0.001
- link Rear_Cover: mass 0.4497186658385477 -> 0.15; geometry collision mesh filename=./meshes/Rear_Cover.stl scale=0.001 0.001 0.001; visual mesh filename=./meshes/Rear_Cover.stl scale=0.001 0.001 0.001
- link Rear_Head_Plate: mass 0.15477666227232548 -> 0.05; geometry collision mesh filename=./meshes/Rear_Head_Plate.stl scale=0.001 0.001 0.001; visual mesh filename=./meshes/Rear_Head_Plate.stl scale=0.001 0.001 0.001
- link Right_Ankle_Cover: mass 0.10517582367621385 -> 0.01; geometry collision mesh filename=./meshes/Right_Ankle_Cover.stl scale=0.001 0.001 0.001; visual mesh filename=./meshes/Right_Ankle_Cover.stl scale=0.001 0.001 0.001
- link Right_Ankle_Motor: geometry collision mesh filename=./meshes/Right_Ankle_Motor.stl scale=0.001 0.001 0.001; visual mesh filename=./meshes/Right_Ankle_Motor.stl scale=0.001 0.001 0.001
- link Right_Cable_Support: mass 0.4093453218387252 -> 0.08; geometry collision mesh filename=./meshes/Right_Cable_Support.stl scale=0.001 0.001 0.001; visual mesh filename=./meshes/Right_Cable_Support.stl scale=0.001 0.001 0.001
- link Right_Ear: mass 0.08364474291031353 -> 0.01; geometry collision mesh filename=./meshes/Right_Ear.stl scale=0.001 0.001 0.001; visual mesh filename=./meshes/Right_Ear.stl scale=0.001 0.001 0.001
- link Right_Eye: mass 0.11621842473165622 -> 0.02; geometry collision mesh filename=./meshes/Right_Eye.stl scale=0.001 0.001 0.001; visual mesh filename=./meshes/Right_Eye.stl scale=0.001 0.001 0.001
- link Right_Foot: mass 1.8791037124906536 -> 0.22; geometry collision mesh filename=./meshes/Right_Foot.stl scale=0.001 0.001 0.001; visual mesh filename=./meshes/Right_Foot.stl scale=0.001 0.001 0.001
- link Right_Foot_Cover: mass 0.27789077678038787 -> 0.02; geometry collision mesh filename=./meshes/Right_Foot_Cover.stl scale=0.001 0.001 0.001; visual mesh filename=./meshes/Right_Foot_Cover.stl scale=0.001 0.001 0.001
- link Right_Foot_Pad: mass 0.8235307524446847 -> 0.08; geometry collision mesh filename=./meshes/Right_Foot_Pad.stl scale=0.001 0.001 0.001; visual mesh filename=./meshes/Right_Foot_Pad.stl scale=0.001 0.001 0.001
- link Right_Front_Cover: mass 0.561072854334117 -> 0.1; geometry collision mesh filename=./meshes/Right_Front_Cover.stl scale=0.001 0.001 0.001; visual mesh filename=./meshes/Right_Front_Cover.stl scale=0.001 0.001 0.001
- link Right_Head_Support: mass 0.15134820645299715 -> 0.04; geometry collision mesh filename=./meshes/Right_Head_Support.stl scale=0.001 0.001 0.001; visual mesh filename=./meshes/Right_Head_Support.stl scale=0.001 0.001 0.001
- link Right_Hip_Bottom_Holder: mass 0.44482107671145044 -> 0.075; geometry collision mesh filename=./meshes/Right_Hip_Bottom_Holder.stl scale=0.001 0.001 0.001; visual mesh filename=./meshes/Right_Hip_Bottom_Holder.stl scale=0.001 0.001 0.001
- link Right_Hip_Pitch_Motor: mass 0.880 -> 0.920; geometry collision mesh filename=./meshes/Right_Hip_Pitch_Motor.stl scale=0.001 0.001 0.001; visual mesh filename=./meshes/Right_Hip_Pitch_Motor.stl scale=0.001 0.001 0.001
- link Right_Hip_Roll_Connector: mass 0.28535016693976095 -> 0.1; geometry collision mesh filename=./meshes/Right_Hip_Roll_Connector.stl scale=0.001 0.001 0.001; visual mesh filename=./meshes/Right_Hip_Roll_Connector.stl scale=0.001 0.001 0.001
- link Right_Hip_Roll_Motor: mass 0.880 -> 0.920; geometry collision mesh filename=./meshes/Right_Hip_Roll_Motor.stl scale=0.001 0.001 0.001; visual mesh filename=./meshes/Right_Hip_Roll_Motor.stl scale=0.001 0.001 0.001
- link Right_Hip_Top_Holder: mass 0.6080984706410996 -> 0.08; geometry collision mesh filename=./meshes/Right_Hip_Top_Holder.stl scale=0.001 0.001 0.001; visual mesh filename=./meshes/Right_Hip_Top_Holder.stl scale=0.001 0.001 0.001
- link Right_Hip_Yaw_Motor: mass 0.880 -> 0.920; geometry collision mesh filename=./meshes/Right_Hip_Yaw_Motor.stl scale=0.001 0.001 0.001; visual mesh filename=./meshes/Right_Hip_Yaw_Motor.stl scale=0.001 0.001 0.001
- link Right_Hip_Yaw_Support: mass 0.8252087483097528 -> 0.08; geometry collision mesh filename=./meshes/Right_Hip_Yaw_Support.stl scale=0.001 0.001 0.001; visual mesh filename=./meshes/Right_Hip_Yaw_Support.stl scale=0.001 0.001 0.001
- link Right_Holder: mass 0.3779808137618351 -> 0.08; geometry collision mesh filename=./meshes/Right_Holder.stl scale=0.001 0.001 0.001; visual mesh filename=./meshes/Right_Holder.stl scale=0.001 0.001 0.001
- link Right_Knee_Motor: mass 0.880 -> 0.920; geometry collision mesh filename=./meshes/Right_Knee_Motor.stl scale=0.001 0.001 0.001; visual mesh filename=./meshes/Right_Knee_Motor.stl scale=0.001 0.001 0.001
- link Right_Lower_Leg: mass 2.86490129434894 -> 0.33; geometry collision mesh filename=./meshes/Right_Lower_Leg.stl scale=0.001 0.001 0.001; visual mesh filename=./meshes/Right_Lower_Leg.stl scale=0.001 0.001 0.001
- link Right_Lower_Leg_Cover: mass 0.36564522610609057 -> 0.057; geometry collision mesh filename=./meshes/Right_Lower_Leg_Cover.stl scale=0.001 0.001 0.001; visual mesh filename=./meshes/Right_Lower_Leg_Cover.stl scale=0.001 0.001 0.001
- link Right_Top_Cover: mass 0.3062644628817641 -> 0.03; geometry collision mesh filename=./meshes/Right_Top_Cover.stl scale=0.001 0.001 0.001; visual mesh filename=./meshes/Right_Top_Cover.stl scale=0.001 0.001 0.001
- link Right_Upper_Leg: mass 4.188552131228702 -> 0.5; geometry collision mesh filename=./meshes/Right_Upper_Leg.stl scale=0.001 0.001 0.001; visual mesh filename=./meshes/Right_Upper_Leg.stl scale=0.001 0.001 0.001
- link Right_Upper_Leg_Cover: mass 0.47108685403507133 -> 0.075; geometry collision mesh filename=./meshes/Right_Upper_Leg_Cover.stl scale=0.001 0.001 0.001; visual mesh filename=./meshes/Right_Upper_Leg_Cover.stl scale=0.001 0.001 0.001
- link Right_Upper_Leg_Detail: mass 0.036788321506523086 -> 0.01; geometry collision mesh filename=./meshes/Right_Upper_Leg_Detail.stl scale=0.001 0.001 0.001; visual mesh filename=./meshes/Right_Upper_Leg_Detail.stl scale=0.001 0.001 0.001
- link Top_Base_Frame: mass 0.8850450859385088 -> 0.15; geometry collision mesh filename=./meshes/Top_Base_Frame.stl scale=0.001 0.001 0.001; visual mesh filename=./meshes/Top_Base_Frame.stl scale=0.001 0.001 0.001
- link base_link: mass 0.6 -> 1; geometry collision mesh filename=./meshes/base_link.stl scale=0.001 0.001 0.001; visual mesh filename=./meshes/base_link.stl scale=0.001 0.001 0.001
- link imu: mass 0.14185490318820562 -> 0.05; geometry collision mesh filename=./meshes/imu.stl scale=0.001 0.001 0.001; visual mesh filename=./meshes/imu.stl scale=0.001 0.001 0.001
- link imu_mount: mass 0.2546845134769666 -> 0.03; geometry collision mesh filename=./meshes/imu_mount.stl scale=0.001 0.001 0.001; visual mesh filename=./meshes/imu_mount.stl scale=0.001 0.001 0.001
Joints:
- joint Head_Pitch: axis 0.0 1.0 0.0 -> (none); limit lower=-1.0471975511965976 upper=0.8726646259971648 effort=6.0 velocity=45.0 -> (none); type revolute -> fixed
- joint Head_Roll: axis -1.0 0.0 0.0 -> (none); limit lower=-0.5235987755982988 upper=0.5235987755982988 effort=6.0 velocity=45.0 -> (none); type revolute -> fixed
- joint Head_Yaw: axis 0.0 0.0 -1.0 -> (none); limit lower=-0.8726646259971648 upper=0.8726646259971648 effort=6.0 velocity=45.0 -> (none); type revolute -> fixed
- joint Left_Ankle: axis -0.0 -1.0 -0.0 -> 0.0 -1.0 0.0
- joint Left_Hip_Pitch: axis -0.0 1.0 -0.0 -> 0.0 -1.0 0.0; limit lower=-0.6981317007977318 upper=1.0471975511965976 effort=60.0 velocity=20.0 -> lower=-1.047 upper=0.698 effort=60.0 velocity=20.0
- joint Left_Hip_Roll: axis 1.0 0.0 -0.0 -> -1.0 0.0 0.0; limit lower=-0.3490658503988659 upper=0.2617993877991494 effort=60.0 velocity=20.0 -> lower=-0.2618 upper=0.349 effort=60.0 velocity=20.0
- joint Left_Knee: axis 0.0 -1.0 0.0 -> 0.0 1.0 0.0; limit lower=-1.3089969389957472 upper=0.9599310885968813 effort=60.0 velocity=20.0 -> lower=-0.9599 upper=1.309 effort=60.0 velocity=20.0
- joint Neck_Pitch: axis 0.0 1.0 -0.0 -> (none); limit lower=-0.3490658503988659 upper=0.8726646259971648 effort=17.0 velocity=43.0 -> (none); type revolute -> fixed
- joint Right_Ankle: axis 0.0 -1.0 0.0 -> 0.0 1.0 0.0; limit lower=-0.785 upper=1.2217304763960306 effort=17.0 velocity=43.0 -> lower=-1.2217 upper=0.785 effort=17.0 velocity=43.0
- joint Right_Hip_Pitch: axis -0.0 -1.0 -0.0 -> 0.0 1.0 0.0; limit lower=-1.0471975511965976 upper=0.6981317007977318 effort=60.0 velocity=20.0 -> lower=-0.698 upper=1.047 effort=60.0 velocity=20.0
- joint Right_Knee: axis -0.0 -1.0 -0.0 -> 0.0 -1.0 0.0
